Commit message: RMPFlow implementation temp

File: configs/isaac_rmpflow/maxlab_ur7e_right/maxlab_ur7e_right.urdf (robot description, URDF)
Before this commit: robot maxlab_ur7e, 13 links, 12 joints
Links:
- added link pinch_center, mass 0.001; visual sphere radius=0.008
Joints:
- added joint tool0_to_pinch_center: type fixed, parent tool0, child pinch_center, origin xyz=0 0 0.165 rpy=0 0 0
