Commit message: updates

File: src/factr_teleop/factr_teleop/urdf/factr_teleop_ur5_gello.urdf (robot description, URDF)
Before this commit: robot robot, 7 links, 6 joints
Links:
- removed link uplink
- added link forearm, mass 0.0857; collision mesh filename=package://assets/b3b_eh.stl; collision mesh filename=package://assets/b3b_eh.stl
- link backlink: mass 0.023 -> 0.08019; geometry collision mesh filename=package://assets/arm_link.stl; collision mesh filename=package://assets/b3b_eh.stl
- link base: mass 0.1 -> 0.289562; geometry collision mesh filename=package://assets/ball_bearing.stl; collision mesh filename=package://assets/base.stl
- link handle: mass 0.023 -> 0.1156; geometry collision mesh filename=package://assets/b3b_eh.stl; collision mesh filename=package://assets/b3b_eh.stl
- link shoulder: mass 0.023 -> 0.224102; geometry collision mesh filename=package://assets/ball_bearing.stl; collision mesh filename=package://assets/dc12_a01_cvr_cable_5.stl
- link wrist: mass 0.023 -> 0.03156; geometry collision mesh filename=package://assets/b3b_eh.stl; collision mesh filename=package://assets/b3b_eh.stl
- link wrist_2: mass 0.023 -> 0.03156; geometry collision mesh filename=package://assets/b3b_eh.stl; collision mesh filename=package://assets/b3b_eh.stl
Joints:
- removed joint base-sho_continuous
- removed joint bl-fl_continuous
- removed joint fl-w1_continuous
- removed joint sho-bl_continuous
- removed joint w1-w2_continuous
- removed joint w2-han_continuous
- added joint backl-frontl: type revolute, parent backlink, child forearm, origin xyz=0.2152 0 -0.014 rpy=3.14159 0 2.39872, axis 0 0 1, limit lower=-3.141592653589793 upper=3.141592653589793 effort=10 velocity=10
- added joint base-sho: type revolute, parent base, child shoulder, origin xyz=-0.157855 -0.398947 -0.0662832 rpy=3.14152 -0.0161707 -0.125228, axis 0 0 1, limit lower=-3.141592653589793 upper=3.141592653589793 effort=10 velocity=10
- added joint frontl-w1: type revolute, parent forearm, child wrist, origin xyz=-0.1961 0 -0.019975 rpy=-3.14159 0 -1.57117, axis 0 0 1, limit lower=-3.141592653589793 upper=3.141592653589793 effort=10 velocity=10
- added joint sho-backl: type revolute, parent shoulder, child backlink, origin xyz=-0.019 0 -0.01775 rpy=1.5708 1.35152 1.5708, axis 0 0 1, limit lower=-3.141592653589793 upper=3.141592653589793 effort=10 velocity=10
- added joint w1-w2: type revolute, parent wrist, child wrist_2, origin xyz=-0 0.0149853 -0.040575 rpy=1.5708 0.0401059 -0, axis 0 0 1, limit lower=-3.141592653589793 upper=3.141592653589793 effort=10 velocity=10
- added joint w2-han: type revolute, parent wrist_2, child handle, origin xyz=0 0.0149853 -0.040575 rpy=1.5708 -0.961422 0, axis 0 0 1, limit lower=-3.141592653589793 upper=3.141592653589793 effort=10 velocity=10
